File: largelad.kicad_pcb (KiCad board)
At the start: 2 copper layers, 297 parts, among them SW1 RotaryEncoder_Switch, U3 YAAJ_WeAct_BlackPill_Part_Like

Commit message: flip diodes and blackpill to the top
Parts:
- D1, D10, D100, D101, D102, D103, D104, D105, D106, D107, D108, D109, D11, D110, D111, D112, D113, D114, D115, D116, D117, D118, D119, D12, D120, D121, D122, D123, D124, D125, D126, D127, D128, D129, D13, D130, D131, D132, D133, D134, D135, D136, D137, D138, D139, D14, D140, D141, D142, D143, D144, D146, D148, D15, D16, D17, D18, D19, D2, D20, D21, D22, D23, D24, D25, D26, D27, D28, D29, D3, D30, D31, D32, D33, D34, D35, D36, D37, D38, D4, D40, D41, D42, D43, D44, D45, D46, D47, D48, D49, D5, D50, D51, D52, D53, D54, D55, D56, D57, D58, D59, D6, D60, D61, D62, D63, D64, D65, D66, D67, D68, D69, D7, D70, D71, D72, D73, D74, D75, D76, D77, D78, D79, D8, D80, D81, D82, D83, D84, D85, D86, D87, D88, D89, D9, D90, D91, D92, D93, D94, D95, D96, D97, D98, D99, U3: moved to F.Cu
- moved U3 16.4 mm to (428.0, 213.2), turned to 90 degrees
- moved D70 2.51 mm to (495.1, 234.2)
- moved D44 0.79 mm to (470.5, 177.0)
- moved MX63 0.22 mm to (324.5, 205.7)

Commit message: connect up the columns
Parts:
- added REF**: 2U, MX_Only:MXOnly-2U-ReversedStabilizers-NoSwitch, F.Cu at (548.5, 234.2)
- added REF**: 2U, MX_Only:MXOnly-2U-ReversedStabilizers-NoSwitch, F.Cu at (548.5, 196.1)
- added REF**: 2U, MX_Only:MXOnly-2U-ReversedStabilizers-NoSwitch, F.Cu at (150.8, 224.6)
- added REF**: 2U, MX_Only:MXOnly-2U-ReversedStabilizers-NoSwitch, F.Cu at (388.9, 224.6)
- added REF**: 6.25U, MX_Only:MXOnly-6.25U-ReversedStabilizers-NoSwitch, F.Cu at (260.4, 243.7)
- added REF**: 2U, MX_Only:MXOnly-2U-ReversedStabilizers-NoSwitch, F.Cu at (396.1, 167.5)
- added REF**: 2U, MX_Only:MXOnly-2U-ReversedStabilizers-NoSwitch, F.Cu at (500.9, 243.7)
- added REF**: 2U, MX_Only:MXOnly-2U-ReversedStabilizers-NoSwitch, F.Cu at (393.7, 205.6)
- D145, D147, D39: moved to F.Cu
Connections:
- SW1 pad A: unconnected-(SW1-PadA) -> ENC0
- SW1 pad B: unconnected-(SW1-PadB) -> ENC1
- SW1 pad C: unconnected-(SW1-PadC) -> ENCG
- U3 pad 17: unconnected-(U3-Pad17) -> ENC1
- U3 pad 19: GND -> ENCG
- U3 pad 26: unconnected-(U3-Pad26) -> ENC0
Routing:
- net COL6: track 0.00 -> 609.0 mm, vias 0 -> 2
- net COL4: track 0.00 -> 595.2 mm, vias 0 -> 2
- net COL5: track 0.00 -> 578.1 mm, vias 0 -> 2
- net COL7: track 0.00 -> 552.3 mm
- net COL0: track 0.00 -> 535.2 mm, vias 0 -> 2
- net COL8: track 0.00 -> 532.2 mm, vias 0 -> 2
- net COL3: track 0.00 -> 506.5 mm, vias 0 -> 2
- net COL11: track 0.00 -> 505.7 mm
- net COL2: track 0.00 -> 505.7 mm, vias 0 -> 2
- net COL1: track 0.00 -> 505.2 mm, vias 0 -> 4
- net COL12: track 0.00 -> 425.4 mm, vias 0 -> 2
- net COL9: track 0.00 -> 412.5 mm, vias 0 -> 2
- net ROW4: track 0.00 -> 365.6 mm
- net ROW5: track 0.00 -> 330.0 mm
- net ROW6: track 0.00 -> 312.3 mm
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
Commit message: route the whole matrix
Parts:
- U3: moved to B.Cu
- moved U3 15.3 mm to (428.2, 197.9), turned to -90 degrees
Connections:
- U3 pad 1: unconnected-(U3-Pad1) -> ROW9
- U3 pad 10: unconnected-(U3-Pad10) -> COL10
- U3 pad 11: unconnected-(U3-Pad11) -> COL8
- U3 pad 12: unconnected-(U3-Pad12) -> ROW2
- U3 pad 13: unconnected-(U3-Pad13) -> ROW0
- U3 pad 14: unconnected-(U3-Pad14) -> ROW1
- U3 pad 15: unconnected-(U3-Pad15) -> ENC0
- U3 pad 16: unconnected-(U3-Pad16) -> COL9
- U3 pad 17: ENC1 -> ROW3
- U3 pad 2: unconnected-(U3-Pad2) -> ROW10
- U3 pad 22: unconnected-(U3-Pad22) -> COL2
- U3 pad 23: unconnected-(U3-Pad23) -> COL3
- U3 pad 24: unconnected-(U3-Pad24) -> COL4
- U3 pad 26: ENC0 -> ENC1
- U3 pad 27: unconnected-(U3-Pad27) -> COL1
- U3 pad 28: unconnected-(U3-Pad28) -> COL0
- U3 pad 29: unconnected-(U3-Pad29) -> ROW5
- U3 pad 3: unconnected-(U3-Pad3) -> ROW11
- U3 pad 30: unconnected-(U3-Pad30) -> ROW4
- U3 pad 31: unconnected-(U3-Pad31) -> COL5
- U3 pad 32: unconnected-(U3-Pad32) -> COL6
- U3 pad 33: unconnected-(U3-Pad33) -> ROW6
- U3 pad 34: unconnected-(U3-Pad34) -> COL7
- U3 pad 35: unconnected-(U3-Pad35) -> ROW7
- U3 pad 37: unconnected-(U3-Pad37) -> ROW8
- U3 pad 4: unconnected-(U3-Pad4) -> COL12
- U3 pad 5: unconnected-(U3-Pad5) -> COL11
Routing:
- net ROW11: track 225.5 -> 451.0 mm, vias 0 -> 2
- net ROW9: track 202.1 -> 413.3 mm, vias 0 -> 1
- net ROW10: track 221.2 -> 421.3 mm, vias 0 -> 2
- net ROW7: track 223.8 -> 413.8 mm, vias 0 -> 1
- net ROW8: track 272.0 -> 443.7 mm, vias 0 -> 3
- net COL12: track 425.4 -> 582.2 mm, vias 2 -> 4
- net COL9: track 412.5 -> 561.1 mm, vias 2 -> 3
- net COL11: track 505.7 -> 638.9 mm, vias 0 -> 2
- net COL10: track 201.2 -> 327.5 mm, vias 0 -> 3
- net COL0: track 535.2 -> 636.7 mm, vias 2 -> 3
- net ROW6: track 312.3 -> 404.2 mm
- net ROW0: track 247.1 -> 330.9 mm, vias 0 -> 1
- net COL8: track 532.2 -> 611.5 mm, vias 2 -> 5
- net COL1: track 505.2 -> 583.6 mm, vias 4 -> 5
- net ROW1: track 247.7 -> 311.0 mm, vias 0 -> 1
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Other:
- board text added: "1"
- board text added: "10"
- board text added: "11"
- board text added: "12"
- board text added: "13"
- board text added: "14"
- board text added: "15"
- board text added: "16"
- board text added: "17"
- board text added: "2"
- board text added: "22"
- board text added: "23"
- board text added: "24"
- board text added: "26"
- board text added: "27"
- board text added: "28"
- board text added: "29"
- board text added: "3"
- board text added: "30"
- board text added: "31"
- board text added: "32"
- board text added: "33"
- board text added: "34"
- board text added: "35"
- board text added: "37"
- board text added: "4"
- board text added: "5"
- board text added: "G"

Commit message: add edge cuts, move some diodes away from stab holes
Parts:
- moved D70 16.0 mm to (480.6, 240.7), turned to 90 degrees
- moved D40 8.47 mm to (535.5, 196.1), turned to 180 degrees
- moved D53 8.23 mm to (535.8, 234.3), turned to 180 degrees
- moved D69 5.64 mm to (480.5, 226.9)
- moved D102 3.71 mm to (152.8, 214.8)
Routing:
- net Net-(D40-Pad2): track 3.51 -> 16.5 mm, vias 0 -> 2
- net Net-(D53-Pad2): track 3.51 -> 15.6 mm
- net ROW3: track 295.0 -> 286.1 mm
- net ROW4: track 383.3 -> 376.9 mm
- net Net-(D70-Pad2): track 10.7 -> 16.1 mm
- net ROW5: track 363.7 -> 369.1 mm
- net Net-(D69-Pad2): track 3.51 -> 4.43 mm
- net COL0: track 636.7 -> 636.0 mm
Other:
- board outline added: 490.5 x 146.8 mm

Commit message: shrink pcb bottom a little
Other:
- board size 490.5 x 146.8 mm -> 490.5 x 144.1 mm
Changed lines of the file:
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@@
     (aux_axis_origin 67.5 109.8)
     (pcbplotparams
-      (layerselection 0x00010fc_ffffffff)
+      (layerselection 0x00010f0_ffffffff)
       (disableapertmacros false)
       (usegerberextensions false)
       (usegerberattributes true)
       (usegerberadvancedattributes true)
-      (creategerberjobfile true)
+      (creategerberjobfile false)
       (svguseinch false)
       (svgprecision 6)
@@
       (plotinvisibletext false)
       (sketchpadsonfab false)
-      (subtractmaskfromsilk false)
+      (subtractmaskfromsilk true)
       (outputformat 1)
       (mirror false)
-      (drillshape 1)
+      (drillshape 0)
       (scaleselection 1)
-      (outputdirectory "")
+      (outputdirectory "gerbers/")
     )
   )
@@
   (gr_line locked (start 550.7858 225.6349) (end 554.0138 225.6349) (layer "Dwgs.User") (width 0.2))
   (gr_arc (start 67.514214 112.364214) (mid 68.1 110.95) (end 69.514214 110.364214) (layer "Edge.Cuts") (width 0.1))
-  (gr_arc (start 557.985786 255.135786) (mid 557.4 256.55) (end 555.985786 257.135786) (layer "Edge.Cuts") (width 0.1))
+  (gr_line (start 67.514216 112.364215) (end 67.514216 251.185782) (layer "Edge.Cuts") (width 0.1))
+  (gr_line (start 67.514216 251.185782) (end 67.514216 252.508) (layer "Edge.Cuts") (width 0.1))
   (gr_arc (start 555.985786 110.364214) (mid 557.4 110.95) (end 557.985786 112.364214) (layer "Edge.Cuts") (width 0.1))
+  (gr_line (start 530.599904 254.508) (end 555.985676 254.508) (layer "Edge.Cuts") (width 0.1))
+  (gr_line (start 69.514216 254.508) (end 71.53 254.508) (layer "Edge.Cuts") (width 0.1))
   (gr_line (start 69.514214 110.364214) (end 555.985786 110.364214) (layer "Edge.Cuts") (width 0.1))
-  (gr_line (start 555.985786 257.135786) (end 69.514214 257.135786) (layer "Edge.Cuts") (width 0.1))
-  (gr_line (start 557.985786 112.364214) (end 557.985786 251.185786) (layer "Edge.Cuts") (width 0.1))
-  (gr_line (start 557.985786 255.135786) (end 557.985786 251.185786) (layer "Edge.Cuts") (width 0.1))
-  (gr_line (start 67.514214 255.135786) (end 67.514214 112.364214) (layer "Edge.Cuts") (width 0.1))
-  (gr_arc (start 69.514214 257.135786) (mid 68.1 256.55) (end 67.514214 255.135786) (layer "Edge.Cuts") (width 0.1))
+  (gr_line (start 530.599904 254.508) (end 71.530007 254.508) (layer "Edge.Cuts") (width 0.1))
+  (gr_line (start 557.985676 112.364215) (end 557.985676 252.508004) (layer "Edge.Cuts") (width 0.1))
+  (gr_arc (start 69.514216 254.508) (mid 68.099998 253.922218) (end 67.514216 252.508) (layer "Edge.Cuts") (width 0.1))
+  (gr_arc (start 557.985676 252.508004) (mid 557.399894 253.922222) (end 555.985676 254.508004) (layer "Edge.Cuts") (width 0.1))
   (gr_text "32" (at 448.55 211.05) (layer "Dwgs.User")
     (effects (font (size 1 1) (thickness 0.15)))
